Commit message: + change controller to id 2 for yaw left and right + modify xacro to use base_footprint

File: bumperbot_ws/src/bumperbot_bringup/urdf/rover.xacro (robot description, xacro)
@@ -21,6 +21,6 @@
     <!-- BASE FOOTPRINT JOINT -->
     <joint name="base_footprint_joint" type="fixed">
-        <parent link="base_link"/>
-        <child link="base_footprint"/>
+        <parent link="base_footprint"/>
+        <child link="base_link"/>
         <origin xyz="0 0 0" rpy="0 0 0"/>
     </joint>
