Commit message: + added imu gazebo - remove inconsistence gazebo color for camera xacro + modify bumperbot_bringup

File: bumperbot_ws/src/bumperbot_bringup/urdf/bumperbot_gazebo.xacro (robot description, xacro)
@@ -4,4 +4,5 @@
     <plugin name="gazebo_ros2_control" filename="libgazebo_ros2_control.so">
         <parameters>$(find bumperbot_bringup)/config/bumperbot_bringup.yaml</parameters>
+        <!-- <parameters>$(find bumperbot_bringup)/config/bumperbot_controllers.yaml</parameters> -->
     </plugin>
 </gazebo>

File: bumperbot_ws/src/bumperbot_bringup/urdf/rover.xacro (robot description, xacro)
@@ -138,5 +138,5 @@
     </link>
     <gazebo reference="camera_link">
-        <material>Gazebo/Blue</material>
+        <material>Gazebo/Black</material>
     </gazebo>
     <joint name="camera_optical_joint" type="fixed">
@@ -199,4 +199,30 @@
         <material>Gazebo/Blue</material>
     </gazebo>
+    <!-- IMU JOINT -->
+    <joint name="imu_joint" type="fixed">
+        <origin xyz="0.0 0.0 0.015 " rpy="0.0 0.0 0.0"/>
+        <parent link="ldlidar_link"/>
+        <child link="imu_link"/>
+    </joint>
+    <!-- IMU LINK -->
+    <link name="imu_link">
+    <visual>
+        <geometry>
+            <cylinder radius="0.01" length="0.01"/>
+        </geometry>
+        <material name="white"/>
+    </visual>
+    <collision>
+        <geometry>
+            <cylinder radius="0.01" length="0.01"/>
+        </geometry>
+    </collision>
+    <xacro:inertial_cylinder mass="0.1" length="0.01" radius="0.01">
+        <origin xyz="0.0 0.0 0.0" rpy="0.0 0.0 0.0"/>
+    </xacro:inertial_cylinder>
+    </link>
+    <gazebo reference="imu_link">
+        <material>Gazebo/White</material>
+    </gazebo>
     <!-- CASTER HOLDER JOINT -->
     <joint name="caster_holder_joint" type="fixed">
@@ -257,5 +283,4 @@
     <!-- GAZEBO Lidar Plugin -->
     <gazebo reference="ldlidar_link">
-        <material>Gazebo/Blue</material>
         <sensor name="laser" type="ray">
             <pose> 0 0 0 0 0 0 </pose>
@@ -296,5 +321,4 @@
     <!-- CAMERA  Plugin -->
     <gazebo reference="camera_link">
-        <material>Gazebo/Black</material>
         <sensor type="camera" name="camera">
         <pose>0 0 0 0 0 0</pose>
@@ -331,3 +355,72 @@
         </sensor>
     </gazebo>
+    <!-- IMU -->
+    <!--Refer to this link https://docs.ros.org/en/rolling/p/gazebo_plugins/generated/classgazebo__plugins_1_1GazeboRosImuSensor.html#class-documentation -->
+    <gazebo reference="imu_link">
+        <sensor name="imu_sensor" type="imu">
+        <!-- ensure the sensor is active (required) -->
+        <always_on>true</always_on>
+        <update_rate>100</update_rate>
+        <plugin name="imu_plugin" filename="libgazebo_ros_imu_sensor.so">
+            <ros>
+            <!-- publish to /imu/out -->
+            <namespace>/imu</namespace>
+            <remapping>~/out:=out</remapping>
+            </ros>
+        </plugin>
+        </sensor>
+        <!--2nd Imu Option-->
+        <!-- <sensor name="imu_sensor" type="imu">
+            <always_on>true</always_on>
+            <update_rate>100</update_rate>
+            <plugin name="my_imu_plugin" filename="libgazebo_ros_imu_sensor.so">
+                <ros>
+                    <namespace>/imu</namespace>
+                    <remapping>~/out:=out</remapping>
+                </ros>
+                <imu>
+                <angular_velocity>
+                    <x>
+                    <noise type="gaussian">
+                        <mean>0.0</mean>
+                        <stddev>2e-4</stddev>
+                    </noise>
+                    </x>
+                    <y>
+                    <noise type="gaussian">
+                        <mean>0.0</mean>
+                        <stddev>2e-4</stddev>
+                    </noise>
+                    </y>
+                    <z>
+                    <noise type="gaussian">
+                        <mean>0.0</mean>
+                        <stddev>2e-4</stddev>
+                    </noise>
+                    </z>
+                </angular_velocity>
+                <linear_acceleration>
+                    <x>
+                    <noise type="gaussian">
+                        <mean>0.0</mean>
+                        <stddev>1.7e-2</stddev>
+                    </noise>
+                    </x>
+                    <y>
+                    <noise type="gaussian">
+                        <mean>0.0</mean>
+                        <stddev>1.7e-2</stddev>
+                    </noise>
+                    </y>
+                    <z>
+                    <noise type="gaussian">
+                        <mean>0.0</mean>
+                        <stddev>1.7e-2</stddev>
+                    </noise>
+                    </z>
+                </linear_acceleration>
+                </imu>
+        </plugin>
+        </sensor> -->
+      </gazebo>
 </robot>
